File: PiZero-RAK.brd (EAGLE design)
At the start: 104.8 x 54.6 mm, 25 parts, among them J1 2.54_I2C, J11 CON_HEADER_1X06-PTH, J2 CONN_20X2HLE, J7 2.54_I2C, J9 2.54_I2C, X1 SPTAF_23.5, X2 SPTAF_25.0MM

Commit message: Bump to V1.3b
Parts:
- JP1: value 5VIN -> JUMPER-PAD-2-NOYES_SILK; device SparkFun-Passives:PAD-JUMPER-2-NC_BY_TRACE_YES_SILK -> SparkFun-Passives:PAD-JUMPER-2-NO_YES_SILK
- moved JP1 8.03 mm to (36.2, 11.4)
- moved J7 5.71 mm to (66.7, 48.9)
- moved U$1 1.27 mm to (54.5, 9.91)
- moved J1 0.63 mm to (66.7, 51.4)
- moved U$3 0.63 mm to (33.0, 11.4), turned to 90 degrees
Connections:
- net 5V: now also JP1.2; no longer JP1.1
- net VIN: now also JP1.1; no longer JP1.2
Routing:
- net VIN: track 44.5 -> 30.0 mm
- net 5V: track 204.7 -> 211.8 mm
- net SDA: track 83.7 -> 87.9 mm
- net 3V3: track 165.8 -> 168.6 mm
Other:
- board text added: "RPI Zero Shield for RAK831 LoraWAN Concentrator V1.3a"
- board text added: "Solder JP1 if you use 5V power and no DC/DC step down"
- board text added: "V1.3a"
- board text removed: "Cut the wire if you plug a DC/DC 5V step down"
- board text removed: "RPI Zero Shield for RAK831 LoraWAN Concentrator V1.3"
- board text removed: "V1.3"

Commit message: Bump to V1.4
Parts:
- added LED3: LED0805, _c2h:0805-LED
- added R1: 390, _c2h:AXIAL-0.4
- added R6: (no value), _c2h:0805-RES
- added U$4: PAD PWR, _c2h:PAD-JUMPER-SWAP
- added U$5: PAD I2C, _c2h:PAD-JUMPER-SWAP
- added U$6: IO4, _c2h:LED3MM
- moved J11 1.27 mm to (90.8, 10.8)
- moved U$9 0.64 mm to (93.3, 34.3)
- renumbered J1 to I2C-2, J7 to I2C-1, J9 to I2C-3
Connections:
- new net N$16: LED3.PLUS, R1.P$2, R6.2, U$6.PLUS
- new net SD$1: I2C-1.4, U$5.3
- new net SD$2: I2C-1.3, U$5.2
- new net V+O: I2C-1.1, U$4.3
- new net V-O: I2C-1.2, U$4.2
- net 3V3: now also U$4.4, U$4.44; no longer I2C-1.1
- net GND: now also LED3.MINUS, U$4.1, U$4.11, U$6.MINUS; no longer I2C-1.2
- net GPIO4: now also R1.P$1, R6.1
- net SCL: now also U$5.1, U$5.11; no longer I2C-1.3
- net SDA: now also U$5.4, U$5.44; no longer I2C-1.4
Routing:
- net GPIO4: track 5.59 -> 34.5 mm
- net N$16: track 0.00 -> 10.7 mm
- net 3V3: track 168.6 -> 177.9 mm, vias 0 -> 1
- net SCL: track 75.1 -> 83.7 mm
- net SD$1: track 0.00 -> 6.68 mm
- net V+O: track 0.00 -> 6.67 mm
- net SD$2: track 0.00 -> 5.23 mm
- net V-O: track 0.00 -> 5.22 mm
- net SDA: track 87.9 -> 92.1 mm
- net GND: track 6.62 -> 8.40 mm, vias 19 -> 22
- net RXD: track 23.3 -> 24.7 mm
- net TXD: track 9.89 -> 11.2 mm
- net 5V: track 211.8 -> 213.1 mm
Other:
- board text added: "I2C-1"
- board text added: "I2C-2"
- board text added: "I2C-3"
- board text added: "RPI Zero Shield for RAK831 LoraWAN Concentrator V1.4"
- board text added: "V1.4"
- board text removed: "I2C"
- board text removed: "RPI Zero Shield for RAK831 LoraWAN Concentrator"
- board text removed: "RPI Zero Shield for RAK831 LoraWAN Concentrator V1.3a"
- board text removed: "V1.3a"

Commit message: Bump to V1.5
Parts:
- removed C6: (no value), _c2h:CAP-PTH-SMALL
- removed L1, L5: WS2812BLONG, _c2h:WS2812B-LONG
- removed L2, L6: WS2812BNOR, _c2h:LED-RGB-THRU
- removed R6: (no value), _c2h:0805-RES
- removed U$6: IO4, _c2h:LED3MM
- added BAT: CR1220, microbuilder:CR1220
- added C3: 3.3uF, _c2h:0805-CAP-LARGEPADS
- added IC1: PCF8523, microbuilder:SOIC8_150MIL
- added J1: CON_HEADER_1X05-PTH, dp_devices:M1X5
- added LED1, LED2: WS2812BLONG, _c2h:WS2812B-LONG
- added LED4: PPS, _c2h:0805-LED-LARGEPADS
- added Q1: CJ2302, Seeed-Transistor:SOT-23
- added R3: 390, _c2h:0805-RES
- added R4: 1K, _c2h:0805-RES
- added SW2: (no value), Seeed-Switch:SW6-2.54-9.0X3.5X3.2+2.0MM
- added Y1: 32.768KHz, adafruit:TC26H
- added Y2: (no value), microbuilder:CRYSTAL_8X3.8
- C4: value (none) -> 10uF; device _c2h:CAP-PTH-SMALL -> _c2h:0805-CAP-LARGEPADS
- LED3: value LED0805 -> IO26; device _c2h:0805-LED -> _c2h:0805-LED-LARGEPADS
- R1: device _c2h:AXIAL-0.4 -> _c2h:0805-RES
- moved LED3 86.7 mm to (21.0, 55.2), turned to 0 degrees
- moved R1 78.2 mm to (25.4, 55.2), turned to 180 degrees
- moved C4 72.8 mm to (41.9, 14.6), turned to 270 degrees
- moved U$1 45.6 mm to (93.2, 34.0)
- moved C2 5.85 mm to (101.0, 20.3), turned to 270 degrees
- moved J11 4.45 mm to (86.4, 10.8)
- moved I2C-3 3.86 mm to (62.9, 11.4)
- moved C1 3.42 mm to (101.0, 47.0), turned to 270 degrees
- moved U$9 1.27 mm to (92.1, 34.3)
Connections:
- removed net N$18: L5.2, L6.4
- removed net N$29: J2.32, U$2.GPIO12/PWM0@32
- removed net RXD: J11.4, J2.10, U$2.GPIO15/RXD@10
- removed net TXD: J11.5, J2.8, U$2.GPIO14/TXD@8
- new net GPIO26: J2.37, R1.1, U$2.GPIO26@37
- new net N$26: IC1.1, Y1.1, Y2.P$4
- new net N$27: Q1.3, R3.1
- new net N$38: IC1.2, Y1.2, Y2.P$1
- new net RXD_PI: J2.10, SW2.COM2, U$2.GPIO15/RXD@10
- new net RX_FTDI: J11.5, SW2.CH1B
- new net RX_GPS: J1.2, SW2.CH1A
- new net SQW: IC1.7, J2.32, U$2.GPIO12/PWM0@32
- new net TXD_PI: J2.8, SW2.COM1, U$2.GPIO14/TXD@8
- new net TX_FTDI: J11.4, SW2.CH2B
- new net TX_GPS: J1.3, SW2.CH2A
- new net VBAT: BAT.+$1, IC1.3
- new net VDD: C3.1, IC1.8, R4.2
- net 3V3: now also C4.1, J1.5, LED4.PLUS, R4.1
- net 5V: now also LED1.1, LED2.1; no longer C4.1, C6.1, L1.1, L2.2, L5.1, L6.2
- net GND: now also BAT.-, C3.2, IC1.4, J1.4, LED1.3, LED2.3, Q1.2; no longer C6.2, L1.3, L2.3, L5.3, L6.3, U$6.MINUS
- net GPIO18: now also LED1.4; no longer L1.4, L2.1
- net GPIO4: now also J1.1, Q1.1; no longer R1.P$1, R6.1
- net N$16: now also R1.2; no longer R1.P$2, R6.2, U$6.PLUS
- net N$37: now also LED4.MINUS, R3.2; no longer J2.37, U$2.GPIO26@37
- net N$39: now also LED1.2, LED2.4; no longer L1.2, L2.4, L5.4, L6.1
- net SCL: now also IC1.6
- net SDA: now also IC1.5
Routing:
- net VBAT: track 0.00 -> 88.2 mm, vias 0 -> 1
- net GPIO26: track 0.00 -> 46.6 mm, vias 0 -> 2
- net N$27: track 0.00 -> 42.8 mm
- net 3V3: track 177.9 -> 215.6 mm, vias 1 -> 2
- net RX_GPS: track 0.00 -> 30.3 mm
- net TX_GPS: track 0.00 -> 25.1 mm
- net RXD: track 24.7 -> 0.00 mm
- net RXD_PI: track 0.00 -> 24.4 mm
- net 5V: track 213.1 -> 191.5 mm
- net RX_FTDI: track 0.00 -> 20.7 mm
- net TX_FTDI: track 0.00 -> 18.9 mm
- net GPIO17: track 113.3 -> 95.1 mm, vias 0 -> 1
- net SCL: track 83.7 -> 101.5 mm
- net TXD_PI: track 0.00 -> 17.3 mm
- net GPIO4: track 34.5 -> 45.8 mm
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Other:
- board text added: "+"
- board text added: "32.768KHz"
- board text added: "Battery is for RTC only"
- board text added: "CJ2302"
- board text added: "FTDI"
- board text added: "GPS"
- board text added: "P"
- board text added: "PPS"
- board text added: "RPI Zero Shield for RAK831 LoraWAN Concentrator V1.5"
- board text added: "RTC"
- board text added: "RXD"
- board text added: "Serial"
- board text added: "TXD"
- board text added: "V1.5"
- board text added: "VIN 36V Max if using DC/DC else 5V"
- board text added: "WS2812B"
- board text added: "Y1"
- board text added: "if 5V power solder JP1 (no DC/DC)"
- board text removed: "Black"
- board text removed: "RPI Zero Shield for RAK831 LoraWAN Concentrator V1.4"
- board text removed: "Solder JP1 if you use 5V power and no DC/DC step down"
- board text removed: "V1.4"
- board text removed: "Vin 36V Max if using DC/DC else 5V only"

Commit message: Bump to V1.5a
Parts:
- added J3, J4: CON_HEADER_1X05-PTH, dp_devices:M1X5
- moved R3 8.98 mm to (89.5, 50.8), turned to 180 degrees
- moved LED4 7.65 mm to (84.5, 50.8)
Connections:
- net 3V3: now also J3.2, J4.2
- net GND: now also J3.1, J4.1
- net SCL: now also J3.4, J4.4
- net SDA: now also J3.3, J4.3
- net SQW: now also J3.5, J4.5
Routing:
- net SQW: track 7.14 -> 55.6 mm, vias 0 -> 2
- net 3V3: track 215.6 -> 254.9 mm
- net SCL: track 101.5 -> 113.2 mm
- net SDA: track 101.8 -> 112.0 mm
- net N$27: track 42.8 -> 32.8 mm
- net GPIO18: track 58.4 -> 55.5 mm
- net MOSI: track 51.1 -> 50.0 mm
- net GPIO17: track 95.1 -> 94.3 mm
Other:
- board text added: "Adafruit RTC"
- board text added: "RPI Zero Shield for RAK831 LoRaWAN Concentrator"
- board text added: "RPI Zero Shield for RAK831 LoRaWAN Concentrator V1.5a"
- board text added: "SQW"
- board text added: "V1.5a"
- board text removed: "RPI Zero Shield for RAK831 LoraWAN Concentrator V1.5"
- board text removed: "V1.5"
